File: SolarMonitor/SolarMonitor_V1/SolarMonitor_V1.kicad_pcb (KiCad board)
At the start: 2 copper layers, 31.5 x 30.5 mm, 38 parts, among them J1 Solar, J2 Battery, J3 Load, J4 Connection1, J5 Connection2, K1 HFD2-003-M-L2-D, K2 HFD2-003-M-L2-D

Commit message: V1 As ordered
Parts:
- removed J3: Load, TerminalBlock:TerminalBlock_bornier-2_P5.08mm
- removed J4: Connection1, TerminalBlock:TerminalBlock_bornier-2_P5.08mm
- removed J5: Connection2, TerminalBlock:TerminalBlock_bornier-2_P5.08mm
- added BRD14: MT3608, stimatofali:MT3608 Boost, F.Cu at (145.9, 74.0)
- BRD2, BRD5: value LM2596 Buck -> ~; footprint stimatofali:LM2596 Module -> stimatofali:MP1584
- J1: value Solar -> Screw_Terminal_01x06; footprint TerminalBlock:TerminalBlock_bornier-2_P5.08mm -> TerminalBlock_RND:TerminalBlock_RND_205-00291_1x06_P5.08mm_Horizontal
- J2: value Battery -> Screw_Terminal_01x04; footprint TerminalBlock:TerminalBlock_bornier-2_P5.08mm -> TerminalBlock_Phoenix:TerminalBlock_Phoenix_MKDS-1,5-4-5.08_1x04_P5.08mm_Horizontal
- moved BRD4 333.7 mm to (137.3, 144.4)
- moved BRD5 319.6 mm to (152.5, 172.5)
- moved BRD6 275.9 mm to (124.3, 143.7), turned to -90 degrees
- moved BRD11 260.7 mm to (113.6, 125.5)
- moved R3 255.2 mm to (99.0, 179.7), turned to 180 degrees
- moved BRD7 244.3 mm to (90.2, 180.8), turned to 180 degrees
- moved R8 241.3 mm to (104.0, 177.2), turned to 180 degrees
- moved R4 239.9 mm to (104.0, 159.0), turned to 180 degrees
- moved R9 235.0 mm to (99.0, 177.2), turned to 180 degrees
- moved R5 233.5 mm to (99.0, 159.0), turned to 180 degrees
- moved R6 225.8 mm to (104.0, 147.0), turned to 180 degrees
- moved R10 220.9 mm to (104.0, 156.0), turned to 180 degrees
- moved R7 219.4 mm to (99.0, 147.0), turned to 180 degrees
- moved R17 217.9 mm to (104.0, 179.7), turned to 180 degrees
- moved R11 214.5 mm to (99.0, 156.0), turned to 180 degrees
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Connections:
- BRD1 pad 1: GND -> Net-(BRD1-OUT+-Pad1)
- BRD1 pad 2: GND -> Net-(BRD1-OUT+-Pad1)
- BRD1 pad 3: Net-(BRD1-OUT+-Pad3) -> GND
- BRD1 pad 4: Net-(BRD1-OUT+-Pad3) -> GND
- BRD1 pad 5: GND -> Net-(BRD1-IN+)
- BRD11 pad 4: /Current Meas & Solar/5V -> /5V
- BRD12 pad 1: /Current Meas & Solar/3V3 -> 3V3
- BRD12 pad 2: /Current Meas & Solar/3V3 -> 3V3
- BRD12 pad 21: /Current Meas & Solar/5V -> /5V
- BRD12 pad 37: /MultiAdd3 -> /MultiAdd0
- BRD12 pad 38: /MultiAdd2 -> /MultiAdd1
- BRD12 pad 39: /MultiAdd1 -> /MultiAdd2
- BRD12 pad 40: /MultiAdd0 -> /MultiAdd3
- BRD13 pad 2: /Current Meas & Solar/3V3 -> 3V3
- BRD2 pad 1: Net-(BRD2-VIN+) -> GND
- BRD2 pad 3: GND -> Net-(BRD2-IN+-Pad3)
- BRD2 pad 4: Net-(BRD2-VOUT+) -> Net-(BRD2-IN+-Pad3)
- BRD4 pad 1: GND -> Net-(BRD4-OUT+-Pad1)
- BRD4 pad 2: GND -> Net-(BRD4-OUT+-Pad1)
- BRD4 pad 3: Net-(BRD4-OUT+-Pad3) -> GND
- BRD4 pad 4: Net-(BRD4-OUT+-Pad3) -> GND
- BRD4 pad 5: GND -> Net-(BRD4-IN+)
- BRD5 pad 1: Net-(BRD5-VIN+) -> GND
- BRD5 pad 3: GND -> Net-(BRD5-IN+-Pad3)
- BRD5 pad 4: Net-(BRD5-VOUT+) -> Net-(BRD5-IN+-Pad3)
- BRD7 pad 23: /3V3 -> 3V3
- BRD8 pad 13: /ExtLoad+ -> Net-(BRD14-VIN+)
- BRD8 pad 8: /Current Meas & Solar/3V3 -> 3V3
- BRD8 pad 9: /Current Meas & Solar/3V3 -> 3V3
- BRD9 pad 14: /Conn2Lo -> /Conn1Lo
- BRD9 pad 16: /Conn1Lo -> /Conn2Lo
- BRD9 pad 8: /Current Meas & Solar/3V3 -> 3V3
- BRD9 pad 9: /Current Meas & Solar/3V3 -> 3V3
- J1 pad 2: /SolarPanel+ -> /ExtLoad+
- J2 pad 1: GND -> /Conn1Hi
- J2 pad 2: /Battery+ -> GND
- K1 pad 11: Net-(BRD2-VIN+) -> Net-(BRD2-IN+-Pad3)
- K1 pad 6: Net-(BRD1-OUT+-Pad3) -> Net-(BRD1-OUT+-Pad1)
- K2 pad 11: Net-(BRD5-VIN+) -> Net-(BRD5-IN+-Pad3)
- K2 pad 6: Net-(BRD4-OUT+-Pad3) -> Net-(BRD4-OUT+-Pad1)
- R17 pad 1: /3V3 -> 3V3
Routing:
- net 3V3: track 67.3 -> 359.1 mm, vias 0 -> 1
- net /Current Meas & Solar/SCL: track 0.00 -> 170.0 mm
- net /Current Meas & Solar/SDA: track 0.00 -> 145.3 mm
- net /ExtLoad+: track 0.00 -> 140.8 mm
- net /5V: track 0.00 -> 131.9 mm
- net /Battery+: track 0.00 -> 129.3 mm
- net /SolarPanel+: track 0.00 -> 120.6 mm
- net GND: track 182.5 -> 73.3 mm, vias 0 -> 8
- net /Conn2Hi: track 0.00 -> 101.3 mm
- net /Conn2Set: track 0.00 -> 95.6 mm
- net /Conn2Reset: track 0.00 -> 93.3 mm
- net /Conn1Set: track 0.00 -> 80.4 mm, vias 0 -> 1
- net /Conn1Reset: track 0.00 -> 80.4 mm, vias 0 -> 1
- net /Current Meas & Solar/SolarPanelHi: track 0.00 -> 71.2 mm
- net /AnaVoutMulti: track 0.00 -> 71.0 mm
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- added copper zone on In1.Cu, net GND
Other:
- board size 31.5 x 30.5 mm -> 140 x 130 mm
- copper layers 2 -> 4
- board text added: "Batt - +"
- board text added: "Ext Load - +"
- board text added: "PWR 1 + -"
- board text added: "PWR 2 + -"
- board text added: "SOLAR - +"
