File: SolarMonitor/SolarMonitor_V1/SolarMonitor_V1.kicad_sch (KiCad schematic)
At the start: 5 parts, among them J1 Solar, J2 Battery, J3 Load, J4 Connection1, J5 Connection2

Commit message: V1 As ordered
Parts:
- removed J1: Solar, TerminalBlock:TerminalBlock_bornier-2_P5.08mm, symbol Connector:Screw_Terminal_01x02
- removed J2: Battery, TerminalBlock:TerminalBlock_bornier-2_P5.08mm, symbol Connector:Screw_Terminal_01x02
- removed J3: Load, TerminalBlock:TerminalBlock_bornier-2_P5.08mm, symbol Connector:Screw_Terminal_01x02
- removed J4: Connection1, TerminalBlock:TerminalBlock_bornier-2_P5.08mm, symbol Connector:Screw_Terminal_01x02
- removed J5: Connection2, TerminalBlock:TerminalBlock_bornier-2_P5.08mm, symbol Connector:Screw_Terminal_01x02
- added J1: Screw_Terminal_01x06, TerminalBlock_RND:TerminalBlock_RND_205-00291_1x06_P5.08mm_Horizontal, symbol Connector:Screw_Terminal_01x06
- added J2: Screw_Terminal_01x04, TerminalBlock_Phoenix:TerminalBlock_Phoenix_MKDS-1,5-4-5.08_1x04_P5.08mm_Horizontal, symbol Connector:Screw_Terminal_01x04
Connections:
- net Battery+: now also J1.4 (Pin_4)
- net Conn1Hi: now also J2.1 (Pin_1)
- net Conn2Hi: now also J2.3 (Pin_3)
- net ExtLoad+: now also J1.2 (Pin_2)
- net GND: now also J1.1 (Pin_1), J1.3 (Pin_3), J1.5 (Pin_5), J2.2 (Pin_2), J2.4 (Pin_4)
- net SolarPanel+: now also J1.6 (Pin_6)
Other:
- sheet Charger1 ports: added 3V3; removed none
- sheet Charger2 ports: added 3V3; removed none
