File: SolarMonitor/SolarMonitor_V1/untitled.kicad_sch (KiCad schematic)
At the start: 2 parts

Commit message: V1 As ordered
Connections:
- net MultiAdd0: now also BRD12.37 (15); no longer BRD12.40 (21)
- net MultiAdd1: now also BRD12.38 (48); no longer BRD12.39 (47)
- net MultiAdd2: now also BRD12.39 (47); no longer BRD12.38 (48)
- net MultiAdd3: now also BRD12.40 (21); no longer BRD12.37 (15)
